File: telakone-aux-gps.brd (EAGLE design)
At the start: 50 x 50 mm, 91 parts, among them X2 MPT0.5/8-2.54, X3 PIIKKIRIMA-3, X4 U.FL-R-SMT-1, X5 PIIKKIRIMA-5, Y1 PTH2.6-5.5SQ, Y2 PTH2.6-5.5SQ, Y3 PTH2.6-5.5SQ, Y4 PTH2.6-5.5SQ

Commit message: routed
Parts:
- moved U$5 55.3 mm to (3.40, 40.9)
- moved R35 13.2 mm to (9.00, 14.5)
- moved R36 9.45 mm to (11.8, 19.3), turned to 270 degrees
- moved C47 7.59 mm to (13.1, 19.3), turned to 90 degrees
- moved D2 5.73 mm to (43.7, 19.0)
- moved C49 5.69 mm to (47.9, 16.7)
- moved R58 5.66 mm to (43.5, 13.8)
- moved R16 4.44 mm to (13.9, 22.4)
- moved R27 3.42 mm to (22.4, 27.6), turned to 270 degrees
- moved V23 2.15 mm to (43.5, 10.3), turned to 0 degrees
- moved C1 2.04 mm to (9.40, 18.5), turned to 270 degrees
- moved C2 2.04 mm to (7.40, 18.5)
- moved C6 2.04 mm to (3.90, 14.5)
- moved C7 2.04 mm to (2.90, 16.5)
- moved L1 2.04 mm to (4.40, 25.0)
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Connections:
- net ACCRTXHI: now also V23.1; no longer V23.2
- net ACCRTXLO: now also V23.2; no longer V23.1
- net IN_CH3: now also V27.3; no longer V27.4
- net IN_CH4: now also V27.4; no longer V27.6
- net IO_CH2: now also V27.6; no longer V27.3
Routing:
- net +3V3: track 0.00 -> 193.9 mm, vias 0 -> 11
- net +12V: track 0.00 -> 59.7 mm, vias 0 -> 1
- net RESETL: track 0.00 -> 56.4 mm, vias 0 -> 1
- net GPS1PPS: track 0.00 -> 41.5 mm
- net OUT1: track 0.00 -> 41.2 mm, vias 0 -> 2
- net MEAS12V: track 0.00 -> 39.4 mm, vias 0 -> 2
- net OUT2: track 0.00 -> 30.7 mm, vias 0 -> 2
- net GND: track 0.00 -> 25.9 mm, vias 0 -> 69
- net IO_CH2: track 0.00 -> 23.7 mm
- net IO_CH1: track 0.00 -> 23.7 mm, vias 0 -> 1
- net SWDIO_CPU: track 0.00 -> 23.6 mm, vias 0 -> 2
- net USART6TX: track 0.00 -> 23.0 mm
- net SWCLK_CPU: track 0.00 -> 21.8 mm, vias 0 -> 2
- net USART6RX: track 0.00 -> 21.8 mm
- net ACCLINKTXE: track 0.00 -> 18.7 mm
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- added copper zone on layer 1, net GND
- added copper zone on layer 16, net GND

Commit message: tuning
Parts:
- removed H6: GRN, omat_ic_2:CHIP-LED0603
- added H2: RED, omat_ic_2:CHIP-LED0603
- added U$1: (no value), dafug:DAFUG
- H4: value RED -> GRN
- moved H4 3.00 mm to (35.5, 47.5)
- renumbered A2 to A1, H5 to H3
Connections:
- net +3V3: now also H4.A; no longer H6.A
- net LED_RED: now also H2.A; no longer H4.A
- net N$3: now also H2.C; no longer H4.C
- net N$5: now also H4.C; no longer H6.C
Routing:
- net N$33: track 0.00 -> 27.2 mm
Other:
- board text added: "+12V"
- board text added: "+3V3"
- board text added: "GND"
- board text added: "IOCH1"
- board text added: "IOCH2"
- board text added: "IOCH3"
- board text added: "IOCH4"
- board text added: "RSTL"
- board text added: "RTXH"
- board text added: "RTXL"
- board text added: "RX"
- board text added: "SWCLK"
- board text added: "SWDIO"
- board text added: "TELAKONE GPS V1.00 KIMMOLI 2016"
- board text added: "TX"

Commit message: bom and gerber pdf, tuning
Parts:
- C7: value 100n 0603 -> 100n
Changed lines of the file:
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@@
 <attribute name="VALUE" x="2.63" y="11.96" size="1.27" layer="27"/>
 </element>
-<element name="C7" library="omat_ic_2" package="C0603" value="100n 0603" x="2.9" y="16.5" smashed="yes">
+<element name="C7" library="omat_ic_2" package="C0603" value="100n" x="2.9" y="16.5" smashed="yes">
 <attribute name="NAME" x="1.465" y="16.265" size="1" layer="25" font="vector" rot="R90"/>
 <attribute name="VALUE" x="2.265" y="14.595" size="0.8128" layer="27"/>
