File: telakone-aux-gps.sch (EAGLE design)
At the start: 91 parts, among them X1 MPT0.5/8-2.54, X2 U.FL-R-SMT-1, X3 PIIKKIRIMA-3, X5 PIIKKIRIMA-5, Y1 PTH2.6-5.5SQ, Y2 PTH2.6-5.5SQ, Y3 PTH2.6-5.5SQ, Y4 PTH2.6-5.5SQ

Commit message: first placement, all on board
Parts:
- removed X6: (no value), omat_ic_2:TE_RUUVILIITIN2
- added X4: U.FL-R-SMT-1, omat_ic_2:U.FL-R-SMT-1
- L1: device omat_ic_2:VLP8040-47U -> omat_ic_2:SRN6045-100M
- X1: value MPT0.5/8-2.54 -> (none); device omat_ic_2:MPT0.5/8-2.54 -> omat_ic_2:TE_RUUVILIITIN2
- X2: value U.FL-R-SMT-1 -> MPT0.5/8-2.54; device omat_ic_2:U.FL-R-SMT-1 -> omat_ic_2:MPT0.5/8-2.54
- renumbered LED2 to H1, N2 to N1
Connections:
- net N$18 renamed VCCRF
- net N$4 renamed N1_SENSE
- removed net N$1: L1.A, N1.PH
- removed net N$16: A2.PPS, H1.A
- removed net N$19: A2.RFIN, L3.1, X2.2
- removed net N$8: F1.1, X6.2
- new net +12V_IN: F1.1, X1.2
- new net GPS1PPS: A2.PPS, D1G$2.PA8, H1.A
- new net GPSRF: A2.RFIN, L3.1, X4.2
- new net N1_PHASE: L1.2, N1.PH
- net +12V: now also X2.1; no longer X1.1
- net +3V3: now also L1.1; no longer L1.B
- net ACCRTXHI: now also X2.7; no longer X1.7
- net ACCRTXLO: now also X2.8; no longer X1.8
- net GND: now also X1.1, X2.6, X4.1, X4.3; no longer X1.6, X2.1, X2.3, X6.1
- net IN_CH3: now also X2.4; no longer X1.4
- net IN_CH4: now also X2.5; no longer X1.5
- net IO_CH1: now also X2.2; no longer X1.2
- net IO_CH2: now also X2.3; no longer X1.3
- net LED_GRN: now also D1G$2.PC8; no longer D1G$2.PB9
- net LED_RED: now also D1G$2.PC9; no longer D1G$2.PB8
Other:
- note added: "TIM1_CH1"
- moved on the sheet: H4, H5, H6, L1, R22, R23, R26

Commit message: routed
Connections:
- net ACCRTXHI: now also V23.1; no longer V23.2
- net ACCRTXLO: now also V23.2; no longer V23.1
- net IN_CH3: now also V27.C1; no longer V27.C2
- net IN_CH4: now also V27.C2; no longer V27.C3
- net IO_CH2: now also V27.C3; no longer V27.C1
Changed lines of the file:
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@@
 </variantdefs>
 <classes>
-<class number="0" name="default" width="0" drill="0">
+<class number="0" name="default" width="0.2" drill="0.3">
 </class>
 <class number="2" name="other" width="0.3" drill="0.3">
 <clearance class="1" value="1"/>
+</class>
+<class number="3" name="supply" width="0.3" drill="0.3">
+</class>
+<class number="4" name="power" width="0.5" drill="0.5">
 </class>
 </classes>
@@
 </segment>
 </net>
-<net name="+3V3" class="0">
+<net name="+3V3" class="3">
 <segment>
 <pinref part="+3V3" gate="G$1" pin="+3V3"/>
@@
 </segment>
 </net>
-<net name="+12V" class="0">
+<net name="+12V" class="4">
 <segment>
 <wire x1="139.7" y1="193.04" x2="139.7" y2="200.66" width="0.1524" layer="91"/>
@@
 </segment>
 </net>
-<net name="+12V_IN" class="0">
+<net name="+12V_IN" class="4">
 <segment>
 <pinref part="X1" gate="G$1" pin="2"/>
@@
 </segment>
 </net>
-<net name="+3V3" class="0">
+<net name="+3V3" class="3">
 <segment>
 <pinref part="D2" gate="G$1" pin="VCC"/>
@@
 <junction x="208.28" y="68.58"/>
 <label x="210.82" y="68.58" size="1.778" layer="95"/>
-<wire x1="208.28" y1="68.58" x2="254" y2="68.58" width="0.1524" layer="91"/>
-<pinref part="V23" gate="G$1" pin="1"/>
-<wire x1="254" y1="63.5" x2="254" y2="68.58" width="0.1524" layer="91"/>
-<wire x1="254" y1="68.58" x2="269.24" y2="68.58" width="0.1524" layer="91"/>
+<wire x1="208.28" y1="68.58" x2="248.92" y2="68.58" width="0.1524" layer="91"/>
+<wire x1="248.92" y1="68.58" x2="269.24" y2="68.58" width="0.1524" layer="91"/>
 <wire x1="269.24" y1="68.58" x2="269.24" y2="121.92" width="0.1524" layer="91"/>
-<junction x="254" y="68.58"/>
 <wire x1="269.24" y1="121.92" x2="294.64" y2="121.92" width="0.1524" layer="91"/>
 <pinref part="X2" gate="G$1" pin="8"/>
+<pinref part="V23" gate="G$1" pin="2"/>
+<wire x1="248.92" y1="63.5" x2="248.92" y2="68.58" width="0.1524" layer="91"/>
+<junction x="248.92" y="68.58"/>
 </segment>
 </net>
@@
 <wire x1="208.28" y1="83.82" x2="231.14" y2="83.82" width="0.1524" layer="91"/>
 <label x="210.82" y="83.82" size="1.778" layer="95"/>
-<wire x1="248.92" y1="71.12" x2="231.14" y2="71.12" width="0.1524" layer="91"/>
 <wire x1="231.14" y1="71.12" x2="231.14" y2="83.82" width="0.1524" layer="91"/>
-<pinref part="V23" gate="G$1" pin="2"/>
-<wire x1="248.92" y1="63.5" x2="248.92" y2="71.12" width="0.1524" layer="91"/>
 <wire x1="294.64" y1="124.46" x2="266.7" y2="124.46" width="0.1524" layer="91"/>
 <wire x1="266.7" y1="124.46" x2="266.7" y2="71.12" width="0.1524" layer="91"/>
-<wire x1="266.7" y1="71.12" x2="248.92" y2="71.12" width="0.1524" layer="91"/>
-<junction x="248.92" y="71.12"/>
+<wire x1="266.7" y1="71.12" x2="254" y2="71.12" width="0.1524" layer="91"/>
 <pinref part="X2" gate="G$1" pin="7"/>
+<pinref part="V23" gate="G$1" pin="1"/>
+<wire x1="254" y1="71.12" x2="231.14" y2="71.12" width="0.1524" layer="91"/>
+<wire x1="254" y1="63.5" x2="254" y2="71.12" width="0.1524" layer="91"/>
+<junction x="254" y="71.12"/>
 </segment>
 </net>
@@
 </segment>
 </net>
-<net name="+12V" class="0">
+<net name="+12V" class="4">
 <segment>
 <wire x1="195.58" y1="233.68" x2="195.58" y2="236.22" width="0.1524" layer="91"/>
@@
 <net name="IO_CH2" class="0">
 <segment>
+<wire x1="294.64" y1="134.62" x2="248.92" y2="134.62" width="0.1524" layer="91"/>
+<label x="256.54" y="134.62" size="1.778" layer="95"/>
+<pinref part="R15" gate="G$1" pin="2"/>
+<pinref part="X2" gate="G$1" pin="3"/>
+<pinref part="V27" gate="G$1" pin="C3"/>
+<wire x1="248.92" y1="134.62" x2="213.36" y2="134.62" width="0.1524" layer="91"/>
+<wire x1="223.52" y1="152.4" x2="248.92" y2="152.4" width="0.1524" layer="91"/>
 <pinref part="V10" gate="G$1" pin="C"/>
 <wire x1="248.92" y1="182.88" x2="231.14" y2="182.88" width="0.1524" layer="91"/>
-<wire x1="294.64" y1="134.62" x2="248.92" y2="134.62" width="0.1524" layer="91"/>
-<wire x1="248.92" y1="134.62" x2="248.92" y2="162.56" width="0.1524" layer="91"/>
-<pinref part="V27" gate="G$1" pin="C1"/>
-<wire x1="248.92" y1="162.56" x2="248.92" y2="182.88" width="0.1524" layer="91"/>
-<wire x1="223.52" y1="162.56" x2="248.92" y2="162.56" width="0.1524" layer="91"/>
-<junction x="248.92" y="162.56"/>
-<label x="256.54" y="134.62" size="1.778" layer="95"/>
-<pinref part="R15" gate="G$1" pin="2"/>
-<wire x1="213.36" y1="134.62" x2="248.92" y2="134.62" width="0.1524" layer="91"/>
+<wire x1="248.92" y1="134.62" x2="248.92" y2="152.4" width="0.1524" layer="91"/>
 <junction x="248.92" y="134.62"/>
-<pinref part="X2" gate="G$1" pin="3"/>
+<wire x1="248.92" y1="152.4" x2="248.92" y2="182.88" width="0.1524" layer="91"/>
+<junction x="248.92" y="152.4"/>
 </segment>
 </net>
@@
 <net name="IN_CH3" class="0">
 <segment>
-<wire x1="294.64" y1="132.08" x2="241.3" y2="132.08" width="0.1524" layer="91"/>
-<pinref part="V27" gate="G$1" pin="C2"/>
-<wire x1="241.3" y1="132.08" x2="213.36" y2="132.08" width="0.1524" layer="91"/>
-<wire x1="223.52" y1="157.48" x2="241.3" y2="157.48" width="0.1524" layer="91"/>
-<wire x1="241.3" y1="157.48" x2="241.3" y2="132.08" width="0.1524" layer="91"/>
-<junction x="241.3" y="132.08"/>
+<wire x1="294.64" y1="132.08" x2="246.38" y2="132.08" width="0.1524" layer="91"/>
 <label x="256.54" y="132.08" size="1.778" layer="95"/>
 <pinref part="X2" gate="G$1" pin="4"/>
 <pinref part="R4" gate="G$1" pin="2"/>
+<pinref part="V27" gate="G$1" pin="C1"/>
+<wire x1="246.38" y1="132.08" x2="213.36" y2="132.08" width="0.1524" layer="91"/>
+<wire x1="223.52" y1="162.56" x2="246.38" y2="162.56" width="0.1524" layer="91"/>
+<wire x1="246.38" y1="162.56" x2="246.38" y2="132.08" width="0.1524" layer="91"/>
+<junction x="246.38" y="132.08"/>
 </segment>
 </net>
 <net name="IN_CH4" class="0">
 <segment>
-<wire x1="294.64" y1="129.54" x2="238.76" y2="129.54" width="0.1524" layer="91"/>
-<pinref part="V27" gate="G$1" pin="C3"/>
-<wire x1="238.76" y1="129.54" x2="213.36" y2="129.54" width="0.1524" layer="91"/>
-<wire x1="223.52" y1="152.4" x2="238.76" y2="152.4" width="0.1524" layer="91"/>
-<wire x1="238.76" y1="152.4" x2="238.76" y2="129.54" width="0.1524" layer="91"/>
-<junction x="238.76" y="129.54"/>
+<wire x1="294.64" y1="129.54" x2="243.84" y2="129.54" width="0.1524" layer="91"/>
 <label x="256.54" y="129.54" size="1.778" layer="95"/>
 <pinref part="X2" gate="G$1" pin="5"/>
 <pinref part="R5" gate="G$1" pin="2"/>
+<wire x1="243.84" y1="129.54" x2="213.36" y2="129.54" width="0.1524" layer="91"/>
+<pinref part="V27" gate="G$1" pin="C2"/>
+<wire x1="223.52" y1="157.48" x2="243.84" y2="157.48" width="0.1524" layer="91"/>
+<wire x1="243.84" y1="157.48" x2="243.84" y2="129.54" width="0.1524" layer="91"/>
+<junction x="243.84" y="129.54"/>
 </segment>
 </net>
@@
 </segment>
 </net>
-<net name="+3V3" class="0">
+<net name="+3V3" class="3">
 <segment>
 <pinref part="C13" gate="G$1" pin="1"/>
@@
 </segment>
 </net>
-<net name="+12V" class="0">
+<net name="+12V" class="4">
 <segment>
 <pinref part="R35" gate="G$1" pin="1"/>
@@
 </segment>
 </net>
-<net name="+3V3" class="0">
+<net name="+3V3" class="3">
 <segment>
 <pinref part="+3V2" gate="G$1" pin="+3V3"/>
@@
 </segment>
 </net>
-<net name="+3V3" class="0">
+<net name="+3V3" class="3">
 <segment>
 <pinref part="A2" gate="G$1" pin="VCC"/>

Commit message: tuning
Parts:
- removed H6: GRN, omat_ic_2:LEDCHIP-LED0603
- added H2: RED, omat_ic_2:LEDCHIP-LED0603
- H4: value RED -> GRN
- renumbered A2 to A1, H5 to H3
Connections:
- net +3V3: now also H4.A; no longer H6.A
- net LED_RED: now also H2.A; no longer H4.A
- net N$3: now also H2.C; no longer H4.C
- net N$5: now also H4.C; no longer H6.C
Other:
- moved on the sheet: H4
Changed lines of the file:
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@@
 </variantdefs>
 <classes>
-<class number="0" name="default" width="0.2" drill="0.3">
+<class number="0" name="default" width="0" drill="0">
 </class>
 <class number="2" name="other" width="0.3" drill="0.3">
@@
 <part name="GND1" library="EKE" deviceset="GND" device=""/>
 <part name="+3V5" library="EKE" deviceset="+3V3" device=""/>
-<part name="A2" library="omat_ic_2" deviceset="UBLOX-NEO6" device=""/>
+<part name="A1" library="omat_ic_2" deviceset="UBLOX-NEO6" device=""/>
 <part name="GND12" library="EKE" deviceset="GND" device=""/>
 <part name="GND13" library="EKE" deviceset="GND" device=""/>
@@
 <part name="C10" library="omat_ic_2" deviceset="CAP" device="0603" value="10n"/>
 <part name="X2" library="omat_ic_2" deviceset="MPT0.5/8-2.54" device=""/>
-<part name="H4" library="omat_ic_2" deviceset="LED" device="CHIP-LED0603" value="RED"/>
-<part name="H5" library="omat_ic_2" deviceset="LED" device="CHIP-LED0603" value="GRN"/>
+<part name="H2" library="omat_ic_2" deviceset="LED" device="CHIP-LED0603" value="RED"/>
+<part name="H3" library="omat_ic_2" deviceset="LED" device="CHIP-LED0603" value="GRN"/>
 <part name="R22" library="omat_ic_2" deviceset="RES" device="0603" value="499"/>
 <part name="R23" library="omat_ic_2" deviceset="RES" device="0603" value="499"/>
 <part name="GND7" library="EKE" deviceset="GND" device=""/>
 <part name="GND20" library="EKE" deviceset="GND" device=""/>
-<part name="H6" library="omat_ic_2" deviceset="LED" device="CHIP-LED0603" value="GRN"/>
+<part name="H4" library="omat_ic_2" deviceset="LED" device="CHIP-LED0603" value="GRN"/>
 <part name="R26" library="omat_ic_2" deviceset="RES" device="0603" value="499"/>
 <part name="GND21" library="EKE" deviceset="GND" device=""/>
@@
 </plain>
 <instances>
-<instance part="H4" gate="G$1" x="289.56" y="172.72"/>
-<instance part="H5" gate="G$1" x="299.72" y="172.72"/>
+<instance part="H2" gate="G$1" x="289.56" y="172.72"/>
+<instance part="H3" gate="G$1" x="299.72" y="172.72"/>
 <instance part="R22" gate="G$1" x="289.56" y="162.56" rot="R90"/>
 <instance part="R23" gate="G$1" x="299.72" y="162.56" rot="R90"/>
 <instance part="GND7" gate="1" x="289.56" y="154.94"/>
 <instance part="GND20" gate="1" x="299.72" y="154.94"/>
-<instance part="H6" gate="G$1" x="279.4" y="172.72"/>
+<instance part="H4" gate="G$1" x="279.4" y="172.72"/>
 <instance part="R26" gate="G$1" x="279.4" y="162.56" rot="R90"/>
 <instance part="GND21" gate="1" x="279.4" y="154.94"/>
@@
 <segment>
 <pinref part="+3V2" gate="G$1" pin="+3V3"/>
-<pinref part="H6" gate="G$1" pin="A"/>
+<pinref part="H4" gate="G$1" pin="A"/>
 <wire x1="279.4" y1="180.34" x2="279.4" y2="175.26" width="0.1524" layer="91"/>
 </segment>
@@
 <segment>
 <pinref part="R23" gate="G$1" pin="2"/>
-<pinref part="H5" gate="G$1" pin="C"/>
+<pinref part="H3" gate="G$1" pin="C"/>
 </segment>
 </net>
 <net name="N$3" class="0">
 <segment>
-<pinref part="H4" gate="G$1" pin="C"/>
+<pinref part="H2" gate="G$1" pin="C"/>
 <pinref part="R22" gate="G$1" pin="2"/>
 </segment>
@@
 <net name="LED_RED" class="0">
 <segment>
-<pinref part="H4" gate="G$1" pin="A"/>
+<pinref part="H2" gate="G$1" pin="A"/>
 <label x="157.48" y="165.1" size="1.778" layer="95"/>
 <wire x1="289.56" y1="175.26" x2="289.56" y2="193.04" width="0.1524" layer="91"/>
@@
 <net name="LED_GRN" class="0">
 <segment>
-<pinref part="H5" gate="G$1" pin="A"/>
+<pinref part="H3" gate="G$1" pin="A"/>
 <label x="157.48" y="162.56" size="1.778" layer="95"/>
 <pinref part="D1" gate="G$2" pin="PC8"/>
@@
 <net name="N$5" class="0">
 <segment>
-<pinref part="H6" gate="G$1" pin="C"/>
+<pinref part="H4" gate="G$1" pin="C"/>
 <pinref part="R26" gate="G$1" pin="2"/>
 </segment>
@@
 </plain>
 <instances>
-<instance part="A2" gate="G$1" x="190.5" y="167.64"/>
+<instance part="A1" gate="G$1" x="190.5" y="167.64"/>
 <instance part="GND12" gate="1" x="167.64" y="137.16"/>
 <instance part="GND13" gate="1" x="223.52" y="139.7"/>
@@
 <net name="GND" class="2">
 <segment>
-<pinref part="A2" gate="G$1" pin="GND1"/>
+<pinref part="A1" gate="G$1" pin="GND1"/>
 <pinref part="GND12" gate="1" pin="GND"/>
 <wire x1="172.72" y1="149.86" x2="167.64" y2="149.86" width="0.1524" layer="91"/>
 <wire x1="167.64" y1="149.86" x2="167.64" y2="144.78" width="0.1524" layer="91"/>
-<pinref part="A2" gate="G$1" pin="GND2"/>
+<pinref part="A1" gate="G$1" pin="GND2"/>
 <wire x1="167.64" y1="144.78" x2="167.64" y2="142.24" width="0.1524" layer="91"/>
 <wire x1="167.64" y1="142.24" x2="167.64" y2="139.7" width="0.1524" layer="91"/>
 <wire x1="172.72" y1="144.78" x2="167.64" y2="144.78" width="0.1524" layer="91"/>
 <junction x="167.64" y="144.78"/>
-<pinref part="A2" gate="G$1" pin="VDDUSB"/>
+<pinref part="A1" gate="G$1" pin="VDDUSB"/>
 <wire x1="172.72" y1="160.02" x2="167.64" y2="160.02" width="0.1524" layer="91"/>
 <wire x1="167.64" y1="160.02" x2="167.64" y2="149.86" width="0.1524" layer="91"/>
@@
 </segment>
 <segment>
-<pinref part="A2" gate="G$1" pin="GND"/>
+<pinref part="A1" gate="G$1" pin="GND"/>
 <pinref part="GND13" gate="1" pin="GND"/>
 <wire x1="218.44" y1="175.26" x2="223.52" y2="175.26" width="0.1524" layer="91"/>
 <wire x1="223.52" y1="175.26" x2="223.52" y2="170.18" width="0.1524" layer="91"/>
-<pinref part="A2" gate="G$1" pin="GND3"/>
+<pinref part="A1" gate="G$1" pin="GND3"/>
 <wire x1="223.52" y1="170.18" x2="223.52" y2="144.78" width="0.1524" layer="91"/>
 <wire x1="223.52" y1="144.78" x2="223.52" y2="142.24" width="0.1524" layer="91"/>
 <wire x1="218.44" y1="144.78" x2="223.52" y2="144.78" width="0.1524" layer="91"/>
 <junction x="223.52" y="144.78"/>
-<pinref part="A2" gate="G$1" pin="VBKUP"/>
+<pinref part="A1" gate="G$1" pin="VBKUP"/>
 <wire x1="218.44" y1="170.18" x2="223.52" y2="170.18" width="0.1524" layer="91"/>
 <junction x="223.52" y="170.18"/>
@@
 <net name="+3V3" class="3">
 <segment>
-<pinref part="A2" gate="G$1" pin="VCC"/>
+<pinref part="A1" gate="G$1" pin="VCC"/>
 <wire x1="218.44" y1="172.72" x2="228.6" y2="172.72" width="0.1524" layer="91"/>
 <wire x1="228.6" y1="172.72" x2="228.6" y2="185.42" width="0.1524" layer="91"/>
@@
 <net name="GPS1PPS" class="0">
 <segment>
-<pinref part="A2" gate="G$1" pin="PPS"/>
+<pinref part="A1" gate="G$1" pin="PPS"/>
 <wire x1="172.72" y1="170.18" x2="162.56" y2="170.18" width="0.1524" layer="91"/>
 <pinref part="H1" gate="G$1" pin="A"/>
@@
 <net name="VCCRF" class="0">
 <segment>
-<pinref part="A2" gate="G$1" pin="VCCRF1"/>
+<pinref part="A1" gate="G$1" pin="VCCRF1"/>
 <wire x1="172.72" y1="154.94" x2="170.18" y2="154.94" width="0.1524" layer="91"/>
-<pinref part="A2" gate="G$1" pin="VCCRF2"/>
+<pinref part="A1" gate="G$1" pin="VCCRF2"/>
 <wire x1="170.18" y1="154.94" x2="160.02" y2="154.94" width="0.1524" layer="91"/>
 <wire x1="172.72" y1="152.4" x2="170.18" y2="152.4" width="0.1524" layer="91"/>
@@
 <net name="GPSRF" class="0">
 <segment>
-<pinref part="A2" gate="G$1" pin="RFIN"/>
+<pinref part="A1" gate="G$1" pin="RFIN"/>
 <pinref part="L3" gate="G$1" pin="1"/>
 <wire x1="134.62" y1="154.94" x2="129.54" y2="154.94" width="0.1524" layer="91"/>
@@
 <net name="GPSRXD" class="0">
 <segment>
-<pinref part="A2" gate="G$1" pin="RXD"/>
+<pinref part="A1" gate="G$1" pin="RXD"/>
 <wire x1="218.44" y1="167.64" x2="261.62" y2="167.64" width="0.1524" layer="91"/>
 <label x="248.92" y="167.64" size="1.778" layer="95"/>
@@
 <net name="GPSTXD" class="0">
 <segment>
-<pinref part="A2" gate="G$1" pin="TXD"/>
+<pinref part="A1" gate="G$1" pin="TXD"/>
 <wire x1="218.44" y1="165.1" x2="261.62" y2="165.1" width="0.1524" layer="91"/>
 <label x="248.92" y="165.1" size="1.778" layer="95"/>
@@
 <net name="N$21" class="0">
 <segment>
-<pinref part="A2" gate="G$1" pin="MOSI/CFGC0"/>
+<pinref part="A1" gate="G$1" pin="MOSI/CFGC0"/>
 <pinref part="R8" gate="G$1" pin="1"/>
 <wire x1="218.44" y1="147.32" x2="228.6" y2="147.32" width="0.1524" layer="91"/>
@@
 <net name="GPSSDA" class="0">
 <segment>
-<pinref part="A2" gate="G$1" pin="SDA"/>
+<pinref part="A1" gate="G$1" pin="SDA"/>
 <wire x1="218.44" y1="160.02" x2="248.92" y2="160.02" width="0.1524" layer="91"/>
 <label x="231.14" y="160.02" size="1.778" layer="95"/>
@@
 <segment>
 <wire x1="251.46" y1="109.22" x2="251.46" y2="162.56" width="0.1524" layer="91"/>
-<pinref part="A2" gate="G$1" pin="SCL"/>
+<pinref part="A1" gate="G$1" pin="SCL"/>
 <wire x1="251.46" y1="162.56" x2="218.44" y2="162.56" width="0.1524" layer="91"/>
 <label x="231.14" y="162.56" size="1.778" layer="95"/>

Commit message: bom and gerber pdf, tuning
Parts:
- C7: value 100n 0603 -> 100n
Changed lines of the file:
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@@
 <part name="GND75" library="EKE" deviceset="GND" device=""/>
 <part name="C6" library="omat_ic_2" deviceset="CAP" device="1206" value="10u 25V 1206"/>
-<part name="C7" library="omat_ic_2" deviceset="CAP" device="0603" value="100n 0603"/>
+<part name="C7" library="omat_ic_2" deviceset="CAP" device="0603" value="100n"/>
 <part name="C1" library="omat_ic_2" deviceset="CAP" device="1206" value="10u 25V 1206"/>
 <part name="C2" library="omat_ic_2" deviceset="CAP" device="1206" value="10u 25V 1206"/>
